File: bt-audio-board.kicad_sch (KiCad schematic)
At the start: 4 parts, among them U1 ESP32-WROOM-32D, U2 MCP73831-2-OT, U3 AMS1117-3.3, U4 WM8960CGEFL_V

Commit message: schematic finished
Parts:
- removed U4: WM8960CGEFL_V, symbol imported:WM8960CGEFL_V
- added BH-18650-B1BA1: ~, imported:BH-18650-B1BA002, symbol imported:BH-18650-B1BA002
- added C1, C12, C13, C14, C2, C7: 4.7u, Capacitor_SMD:C_0603_1608Metric, symbol Device:C_Small
- added C10, C11, C5, C9: 0.1u, Capacitor_SMD:C_0603_1608Metric, symbol Device:C_Small
- added C15, C16: 100u, Capacitor_SMD:CP_Elec_6.3x5.4_Nichicon, symbol Device:C_Polarized_Small
- added C3, C8: 10u, Capacitor_SMD:C_0603_1608Metric, symbol Device:C_Small
- added C4: 22u, Capacitor_SMD:C_0603_1608Metric, symbol Device:C_Small
- added D1: LED, LED_SMD:LED_0603_1608Metric, symbol Device:LED
- added D2: SS34, imported:SS34, symbol imported:SS34
- added D3: 1N5819WS, Diode_SMD:D_SOD-323, symbol Diode:1N5819WS
- added J1: USB_C_Receptacle_PowerOnly_6P, symbol Connector:USB_C_Receptacle_PowerOnly_6P
- added J2: Conn_01x12_Pin, Connector_PinHeader_2.54mm:PinHeader_1x12_P2.54mm_Vertical, symbol Connector:Conn_01x12_Pin
- added PJ-326-3A1: ~, imported:PJ-326-3A, symbol imported:PJ-326-3A
- added R1, R11, R9: 470, Resistor_SMD:R_0603_1608Metric, symbol Device:R_Small
- added R10, R12, R13, R14: 10k, Resistor_SMD:R_0603_1608Metric, symbol Device:R_Small
- added R2: 2k, Resistor_SMD:R_0603_1608Metric, symbol Device:R_Small
- added R3, R4: 5k1, Resistor_SMD:R_0603_1608Metric, symbol Device:R_Small
- added R5, R6, R7, R8: 100, Resistor_SMD:R_0603_1608Metric, symbol Device:R_Small
- added TS5220A1, TS5220A2: ~, imported:TS5220A, symbol imported:TS5220A
- added U4: WM8960CGEFL/V, WM8960CGEFL/V_CIR, symbol 2024-02-02_21-49-10:WM8960CGEFL_V
Connections:
- net GND: now reaches U1.1 (GND), U1.15 (GND), U1.38 (GND), U1.39 (GND)
- net GND: now also U2.2 (V_{SS}), U3.1 (GND), BH-18650-B1BA1.1, C1.2, C10.1, C11.2, C12.2, C13.2, C14.2, C2.2, C3.2, C4.2, C5.2, C7.1, C8.2, C9.1, J1.A12 (GND), J1.B12 (GND), J1.S1 (SHIELD), J2.11 (Pin_11), PJ-326-3A1.1, R2.1, R3.2, R4.2, TS5220A1.3, TS5220A2.3, U4.20 (SPKGND2), U4.24 (SPKGND1), U4.28 (AGND), U4.9 (DGND)
- net I2S_DATA: now reaches U1.10 (IO25)
- net I2S_DATA: now also U4.14 (DACDAT)
- net I2S_BCK: now reaches U1.11 (IO26)
- net I2S_BCK: now also U4.12 (BCLK)
- net at U1.13 (IO14): now also R7.1
- net at U1.14 (IO12): now also R5.2
- net at U1.16 (IO13): now also R6.1
- net VCC: now reaches U1.2 (VDD)
- net VCC: now also U3.2 (VO), C10.2, C11.1, C12.1, C13.1, C14.1, C4.1, C5.1, C7.2, C8.1, C9.2, J2.12 (Pin_12), R10.1, R12.1, R13.1, R14.1, U4.1 (MICBIAS), U4.10 (DBVDD), U4.21 (SPKVDD2), U4.26 (SPKVDD1), U4.27 (VMID), U4.32 (AVDD), U4.8 (DCVDD)
- net at U1.21 (SDO/SD0): now also R13.2
- net at U1.23 (IO15): now also R8.1
- net at U1.3 (EN): now also R14.2
- net SDA: now reaches U1.33 (IO21)
- net SDA: now also J2.6 (Pin_6), U4.18 (SDIN)
- net RX: now reaches U1.34 (RXD0/IO3)
- net TX: now reaches U1.35 (TXD0/IO1)
- net SCL: now reaches U1.36 (IO22)
- net SCL: now also J2.5 (Pin_5), U4.17 (SCLK)
- net I2S_LRCK: now reaches U1.37 (IO23)
- net I2S_LRCK: now also U4.13 (DACLRC)
- net IO32: now reaches U1.8 (IO32)
- net IO32: now also J2.2 (Pin_2), R10.2, R9.1
- net IO33: now reaches U1.9 (IO33)
- net IO33: now also J2.1 (Pin_1), R11.1, R12.2
- net at U2.1 (STAT): now also R1.1
- net at U2.3 (V_{BAT}): now also BH-18650-B1BA1.2, C2.1, D2.2 (A)
- net +5V: now reaches U2.4 (V_{DD})
- net +5V: now also C1.1, D1.2 (A), D3.1 (K)
- net at U2.5 (PROG): now also R2.2
- net at U3.3 (VI): now also C3.1, D2.1 (K)
- new net: J1.A5 (CC1), R4.1
- new net: R9.2, TS5220A1.1
- new net: D1.1 (K), R1.2
- new net: R11.2, TS5220A2.1
- new net: C16.1, U4.29 (HP_R)
- new net: C15.1, U4.31 (HP_L)
- new net: J1.B5 (CC2), R3.1
- new net: D3.2 (A), J1.A9 (VBUS), J1.B9 (VBUS)
- new net EP: J2.3 (Pin_3), U4.33 (EP)
- new net HP_L: C15.2, PJ-326-3A1.2
- new net HP_R: C16.2, PJ-326-3A1.3
- new net MCLK: J2.4 (Pin_4), U4.11 (MCLK)
- new net TCK: J2.9 (Pin_9), R6.2
- new net TDI: J2.10 (Pin_10), R5.1
- new net TDO: J2.7 (Pin_7), R8.2
- new net TMS: J2.8 (Pin_8), R7.2
Other:
- moved on the sheet: U1, U2, U3
